File: magic.sch (EAGLE design)
At the start: 30 parts

Commit message: transformer
Parts:
- removed U$1: PJ-036AH-SMT, magic:PJ-036AH-SMT
- added TRANSFORMER: RAC04-09SC, magic:RAC04-09SC
Connections:
- removed net N$3: SSR.OUT1, U$3.P$1
- removed net N$4: SSR.OUT2, U$2.P$1
- new net VAC(L): SSR.OUT1, TRANSFORMER.VAC(L), U$3.P$1
- new net VAC(N): SSR.OUT2, TRANSFORMER.VAC(N), U$2.P$1
- net GND: now also TRANSFORMER.VDC-; no longer U$1.P$1, U$1.P$2
- net N$1: now also TRANSFORMER.VDC+; no longer U$1.P$3
Changed lines of the file:
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@@
 <part name="R1" library="rcl" library_urn="urn:adsk.eagle:library:334" deviceset="R-US_" device="M1206" package3d_urn="urn:adsk.eagle:package:23566/2" value="1k"/>
 <part name="R2" library="rcl" library_urn="urn:adsk.eagle:library:334" deviceset="R-US_" device="M1206" package3d_urn="urn:adsk.eagle:package:23566/2" value="1k"/>
-<part name="U$1" library="magic" deviceset="PJ-036AH-SMT" device=""/>
 <part name="DIODE" library="magic" deviceset="S1G" device="" package3d_urn="urn:adsk.eagle:package:12434192/1"/>
 <part name="THERMO" library="magic" deviceset="PC6-16/2-G1-10,16" device=""/>
 <part name="U$2" library="magic" deviceset="6-GAUGE" device=""/>
 <part name="U$3" library="magic" deviceset="6-GAUGE" device=""/>
+<part name="TRANSFORMER" library="magic" deviceset="RAC04-09SC" device=""/>
 </parts>
 <sheets>
@@
 <attribute name="VALUE" x="-143.002" y="67.31" size="1.778" layer="96" rot="R270"/>
 </instance>
-<instance part="U$1" gate="G$1" x="-177.8" y="48.26" smashed="yes">
-<attribute name="NAME" x="-185.42" y="58.42" size="1.27" layer="95"/>
-<attribute name="VALUE" x="-185.42" y="40.64" size="1.27" layer="96"/>
-</instance>
 <instance part="DIODE" gate="G$1" x="-165.1" y="53.34" smashed="yes">
 <attribute name="NAME" x="-170.18" y="55.88" size="1.778" layer="95"/>
@@
 <instance part="U$2" gate="G$1" x="-119.38" y="48.26" smashed="yes" rot="R270"/>
 <instance part="U$3" gate="G$1" x="-119.38" y="53.34" smashed="yes" rot="R270"/>
+<instance part="TRANSFORMER" gate="G$1" x="-190.5" y="55.88" smashed="yes"/>
 </instances>
 <busses>
@@
 </segment>
 <segment>
-<pinref part="U$1" gate="G$1" pin="P$2"/>
-<pinref part="U$1" gate="G$1" pin="P$1"/>
-<wire x1="-172.72" y1="48.26" x2="-172.72" y2="45.72" width="0.1524" layer="91"/>
-<wire x1="-172.72" y1="45.72" x2="-167.64" y2="45.72" width="0.1524" layer="91"/>
-<junction x="-172.72" y="45.72"/>
-<label x="-170.18" y="45.72" size="1.778" layer="95"/>
+<pinref part="TRANSFORMER" gate="G$1" pin="VDC-"/>
+<wire x1="-175.26" y1="58.42" x2="-172.72" y2="58.42" width="0.1524" layer="91"/>
+<label x="-175.26" y="58.42" size="1.778" layer="95"/>
 </segment>
 </net>
@@
 <net name="N$1" class="0">
 <segment>
-<pinref part="U$1" gate="G$1" pin="P$3"/>
-<wire x1="-172.72" y1="53.34" x2="-170.18" y2="53.34" width="0.1524" layer="91"/>
 <pinref part="DIODE" gate="G$1" pin="P$1"/>
+<pinref part="TRANSFORMER" gate="G$1" pin="VDC+"/>
+<wire x1="-175.26" y1="53.34" x2="-170.18" y2="53.34" width="0.1524" layer="91"/>
 </segment>
 </net>
@@
 </segment>
 </net>
-<net name="N$3" class="0">
+<net name="VAC(L)" class="0">
 <segment>
 <pinref part="U$3" gate="G$1" pin="P$1"/>
 <pinref part="SSR" gate="G$1" pin="OUT1"/>
 <wire x1="-114.3" y1="53.34" x2="-99.06" y2="53.34" width="0.1524" layer="91"/>
-</segment>
-</net>
-<net name="N$4" class="0">
+<label x="-109.22" y="53.34" size="1.778" layer="95"/>
+</segment>
+<segment>
+<pinref part="TRANSFORMER" gate="G$1" pin="VAC(L)"/>
+<wire x1="-205.74" y1="58.42" x2="-210.82" y2="58.42" width="0.1524" layer="91"/>
+<label x="-218.44" y="58.42" size="1.778" layer="95"/>
+</segment>
+</net>
+<net name="VAC(N)" class="0">
 <segment>
 <pinref part="U$2" gate="G$1" pin="P$1"/>
 <pinref part="SSR" gate="G$1" pin="OUT2"/>
 <wire x1="-114.3" y1="48.26" x2="-99.06" y2="48.26" width="0.1524" layer="91"/>
-</segment>
-</net>
+<label x="-109.22" y="48.26" size="1.778" layer="95"/>
+</segment>
+<segment>
+<pinref part="TRANSFORMER" gate="G$1" pin="VAC(N)"/>
+<wire x1="-205.74" y1="53.34" x2="-210.82" y2="53.34" width="0.1524" layer="91"/>
+<label x="-218.44" y="53.34" size="1.778" layer="95"/>
+</segment>
+</net>

Commit message: redid the board
Parts:
- removed U$2, U$3: 6-GAUGE, magic:6-GAUGE
- added 110VAC(L)_OUT, 110VAC(N)_OUT, AC(L)_IN, AC(N)_IN: 6-GAUGE, magic:6-GAUGE
- added R3, R5: 100, resistor-power:RMG100-V
- added R4, R6: 1k, resistor-power:RMG100-V
Connections:
- new net 10VAC(L): R3.1, R4.2, TRANSFORMER.VAC(L)
- new net 10VAC(N): R5.1, R6.2, TRANSFORMER.VAC(N)
- new net 110VAC(L): R3.2, SSR.OUT1
- new net 110VAC(L)_OUT: 110VAC(L)_OUT.P$1, SSR.OUT2
- new net 110VAC(N): 110VAC(N)_OUT.P$1, R5.2
- net VAC(L): now also AC(L)_IN.P$1, R4.1; no longer SSR.OUT1, TRANSFORMER.VAC(L), U$3.P$1
- net VAC(N): now also AC(N)_IN.P$1, R6.1; no longer SSR.OUT2, TRANSFORMER.VAC(N), U$2.P$1
