File: magic.brd (EAGLE design)
At the start: 113 x 89.8 mm, 29 parts

Commit message: thermocouple block
Parts:
- removed T+, T-: 350180, magic:350180
- added THERMO: PC6-16/2-G1-10,16, magic:PC6-16/2-G1-10,16
- added U$2, U$3: 6-GAUGE, magic:6-GAUGE
Connections:
- removed net AC1: SSR.P$1
- removed net AC2: SSR.P$2
- new net N$3: SSR.P$1, U$3.P$1
- new net N$4: SSR.P$2, U$2.P$1
- net T+: now also THERMO.P$1; no longer T+.P$3
- net T-: now also THERMO.P$2; no longer T-.P$3
Routing:
- net GND: track 484.8 -> 0.00 mm, vias 18 -> 0
- net +5V: track 320.1 -> 0.00 mm, vias 12 -> 0
- net BIT1_: track 252.3 -> 0.00 mm, vias 7 -> 0
- net BIT0: track 235.7 -> 0.00 mm, vias 8 -> 0
- net BIT2: track 202.2 -> 0.00 mm, vias 7 -> 0
- net BIT2_: track 193.8 -> 0.00 mm, vias 8 -> 0
- net BIT3_: track 187.2 -> 0.00 mm, vias 2 -> 0
- net BIT1: track 185.3 -> 0.00 mm, vias 7 -> 0
- net D3A: track 165.3 -> 0.00 mm, vias 2 -> 0
- net BIT0_: track 159.8 -> 0.00 mm, vias 9 -> 0
- net D: track 147.2 -> 0.00 mm, vias 4 -> 0
- net BIT3: track 144.4 -> 0.00 mm, vias 6 -> 0
- net SEL1: track 144.1 -> 0.00 mm, vias 4 -> 0
- net D3: track 126.7 -> 0.00 mm, vias 2 -> 0
- net G: track 122.3 -> 0.00 mm, vias 2 -> 0
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
Commit message: transformer
Parts:
- removed U$1: PJ-036AH-SMT, magic:PJ-036AH-SMT
- added TRANSFORMER: RAC04-09SC, magic:RAC04-09SC
- moved U$3 137.7 mm to (57.1, 25.4)
- moved U$2 136.0 mm to (57.1, 36.2)
- moved 2INOR1 99.7 mm to (-68.6, -12.1)
- moved 2INAND2 88.4 mm to (85.1, 24.8)
- moved 2INOR3 81.6 mm to (-43.2, 54.6)
- moved MUXC/D 73.0 mm to (-64.1, 36.2)
- moved INV 71.1 mm to (-61.6, 5.08)
- moved 4INAND1 61.9 mm to (112.4, -48.3)
- moved MUXG 61.8 mm to (-21.0, -38.7)
- moved MUXE/F 60.4 mm to (-35.6, -28.6)
- moved ARDUINO 58.4 mm to (-43.8, 20.3)
- moved 2INOR2 58.1 mm to (-5.08, 48.9)
- moved 4INOR1 58.0 mm to (82.5, -58.4)
- moved 4INAND2 41.2 mm to (88.3, -5.71)
- moved 3INOR1 39.9 mm to (62.2, 54.6), turned to 90 degrees
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Connections:
- removed net N$3: SSR.P$1, U$3.P$1
- removed net N$4: SSR.P$2, U$2.P$1
- new net VAC(L): SSR.P$1, TRANSFORMER.P$1, U$3.P$1
- new net VAC(N): SSR.P$2, TRANSFORMER.P$3, U$2.P$1
- net GND: now also TRANSFORMER.P$14; no longer U$1.P$1, U$1.P$2
- net N$1: now also TRANSFORMER.P$16; no longer U$1.P$3
- net T-: now also THERMO.P$6; no longer THERMO.P$2
Routing:
- added copper zone on layer 1, net GND
- added copper zone on layer 16, net GND
Other:
- board text added: "2/4/20"
- board text removed: "9/4/19"

Commit message: redid the board
Parts:
- added 110VAC(L)_OUT, 110VAC(N)_OUT: 6-GAUGE, magic:6-GAUGE
- added R3, R5: 100, resistor-power:TO-247-2V
- added R4, R6: 1k, resistor-power:TO-247-2V
- moved 3INOR1 135.2 mm to (-32.4, -41.9), turned to 270 degrees
- moved 3INOR2 127.0 mm to (-42.5, -41.9)
- moved 2INAND2 125.8 mm to (-21.6, -41.9), turned to 270 degrees
- moved 4INAND1 124.2 mm to (-10.8, -32.4)
- moved 3INOR3 122.0 mm to (-42.5, -32.4), turned to 90 degrees
- moved MUXC/D 121.6 mm to (38.7, -28.6)
- moved 4INOR1 117.8 mm to (-32.4, -32.4), turned to 270 degrees
- moved 2INOR3 111.8 mm to (13.3, -41.9), turned to 270 degrees
- moved 4INAND2 111.3 mm to (-21.6, -23.5), turned to 270 degrees
- moved 2INOR2 91.0 mm to (0.64, -41.9), turned to 270 degrees
- moved THERMOCOUPLE 89.7 mm to (-41.9, 11.4), turned to 90 degrees
- moved MUXA/B 83.1 mm to (26.7, -28.6)
- moved 3INAND1 77.1 mm to (-21.6, -32.4), turned to 270 degrees
- moved MUXE/F 49.7 mm to (14.0, -32.4)
- moved 2INAND1 47.5 mm to (-10.8, -41.9), turned to 270 degrees
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- renumbered U$2 to AC(N)_IN, U$3 to AC(L)_IN
Connections:
- new net 10VAC(L): R3.1, R4.2, TRANSFORMER.P$1
- new net 10VAC(N): R5.1, R6.2, TRANSFORMER.P$3
- new net 110VAC(L): R3.2, SSR.P$1
- new net 110VAC(L)_OUT: 110VAC(L)_OUT.P$1, SSR.P$2
- new net 110VAC(N): 110VAC(N)_OUT.P$1, R5.2
- net VAC(L): now also R4.1; no longer SSR.P$1, TRANSFORMER.P$1
- net VAC(N): now also R6.1; no longer SSR.P$2, TRANSFORMER.P$3
Routing:
- net +5V: track 0.00 -> 426.9 mm, vias 0 -> 1
- net BIT1_: track 0.00 -> 163.3 mm, vias 0 -> 13
- net BIT1: track 0.00 -> 162.7 mm, vias 0 -> 7
- net BIT2: track 0.00 -> 153.0 mm, vias 0 -> 8
- net BIT0: track 0.00 -> 148.6 mm, vias 0 -> 6
- net BIT0_: track 0.00 -> 132.0 mm, vias 0 -> 10
- net SEL0: track 0.00 -> 130.3 mm, vias 0 -> 10
- net RELAY: track 0.00 -> 130.2 mm, vias 0 -> 1
- net BIT2_: track 0.00 -> 129.2 mm, vias 0 -> 8
- net SEL1: track 0.00 -> 126.5 mm, vias 0 -> 8
- net BIT3_: track 0.00 -> 108.8 mm, vias 0 -> 5
- net OVER: track 0.00 -> 99.0 mm, vias 0 -> 3
- net BASELINE_CNTRLR: track 0.00 -> 97.8 mm, vias 0 -> 1
- net C: track 0.00 -> 96.6 mm, vias 0 -> 2
- net X: track 0.00 -> 94.7 mm, vias 0 -> 3
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
Commit message: widened AC traces for 1oz copper and made gerber files
Routing:
- net 110VAC(L): track 43.8 -> 51.7 mm
- net 110VAC(N): track 12.1 -> 10.6 mm
- net 10VAC(N): track 40.2 -> 41.3 mm
Changed lines of the file:
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@@
 <setting verticaltext="up"/>
 </settings>
-<grid distance="15" unitdist="mil" unit="mil" style="lines" multiple="1" display="yes" altdistance="1.5" altunitdist="mil" altunit="mil"/>
+<grid distance="50" unitdist="mil" unit="mil" style="lines" multiple="1" display="yes" altdistance="5" altunitdist="mil" altunit="mil"/>
 <layers>
 <layer number="1" name="Top" color="4" fill="1" visible="yes" active="yes"/>
@@
 </class>
 </classes>
-<designrules name="default">
+<designrules name="default *">
 <description language="de">&lt;b&gt;EAGLE Design Rules&lt;/b&gt;
 &lt;p&gt;
@@
 </element>
 <element name="DIODE" library="magic" package="S1G" package3d_urn="urn:adsk.eagle:package:12434192/1" value="S1G" x="-34.925" y="39.37" smashed="yes">
-<attribute name="NAME" x="-34.925" y="41.48" size="1.27" layer="25" align="bottom-center"/>
+<attribute name="NAME" x="-28.575" y="38.94" size="1.27" layer="25" align="bottom-center"/>
 <attribute name="VALUE" x="-34.925" y="37.26" size="1.27" layer="27" align="top-center"/>
 </element>
@@
 <contactref element="R4" pad="1"/>
 <contactref element="AC(L)_IN" pad="P$1"/>
-<wire x1="60.96" y1="7.62" x2="60.7382125" y2="7.62" width="1.397" layer="1"/>
-<wire x1="60.7382125" y1="7.62" x2="56.8391" y2="11.5191125" width="1.397" layer="1"/>
-<wire x1="57.15" y1="25.4" x2="56.8391" y2="25.0891" width="1.397" layer="1"/>
-<wire x1="56.8391" y1="25.0891" x2="56.8391" y2="11.5191125" width="1.397" layer="1"/>
+<wire x1="60.96" y1="7.62" x2="57.15" y2="11.43" width="2.7686" layer="1"/>
+<wire x1="57.15" y1="11.43" x2="57.15" y2="25.4" width="2.7686" layer="1"/>
 </signal>
 <signal name="VAC(N)">
 <contactref element="AC(N)_IN" pad="P$1"/>
 <contactref element="R6" pad="1"/>
-<wire x1="60.96" y1="19.10164375" x2="60.96" y2="14.605" width="1.397" layer="1"/>
-<wire x1="62.7709" y1="20.91254375" x2="60.96" y2="19.10164375" width="1.397" layer="1"/>
-<wire x1="57.15" y1="36.195" x2="62.7709" y2="30.5741" width="1.397" layer="1"/>
-<wire x1="62.7709" y1="30.5741" x2="62.7709" y2="20.91254375" width="1.397" layer="1"/>
+<wire x1="60.96" y1="14.605" x2="60.96" y2="20.036775" width="2.7686" layer="1"/>
+<wire x1="60.96" y1="20.036775" x2="62.1867" y2="21.263475" width="2.7686" layer="1"/>
+<wire x1="62.1867" y1="21.263475" x2="62.1867" y2="31.1583" width="2.7686" layer="1"/>
+<wire x1="62.1867" y1="31.1583" x2="57.15" y2="36.195" width="2.7686" layer="1"/>
 </signal>
 <signal name="10VAC(L)">
@@
 <contactref element="R3" pad="1"/>
 <contactref element="TRANSFORMER" pad="P$1"/>
-<wire x1="47.625" y1="20.955" x2="47.625" y2="10.795" width="1.397" layer="16"/>
-<wire x1="47.625" y1="10.795" x2="50.8" y2="7.62" width="1.397" layer="16"/>
-<wire x1="50.8" y1="7.62" x2="50.8" y2="-1.27" width="1.397" layer="16"/>
+<wire x1="47.625" y1="20.955" x2="47.625" y2="16.43165" width="2.7686" layer="16"/>
+<wire x1="47.625" y1="16.43165" x2="47.2633" y2="16.06995" width="2.7686" layer="16"/>
+<wire x1="47.2633" y1="16.06995" x2="47.2633" y2="11.1567" width="2.7686" layer="16"/>
+<wire x1="47.2633" y1="11.1567" x2="50.8" y2="7.62" width="2.7686" layer="16"/>
+<wire x1="50.8" y1="7.62" x2="50.8" y2="-1.27" width="2.7686" layer="16"/>
 </signal>
 <signal name="110VAC(L)">
 <contactref element="R3" pad="2"/>
 <contactref element="SSR" pad="P$1"/>
-<wire x1="56.8391" y1="-7.7091125" x2="56.8391" y2="-11.3408875" width="1.397" layer="16"/>
-<wire x1="60.96" y1="-1.27" x2="60.96" y2="-3.5882125" width="1.397" layer="16"/>
-<wire x1="60.96" y1="-3.5882125" x2="56.8391" y2="-7.7091125" width="1.397" layer="16"/>
-<wire x1="56.8391" y1="-11.3408875" x2="61.5009" y2="-16.0026875" width="1.397" layer="16"/>
-<wire x1="61.5009" y1="-16.0026875" x2="61.5009" y2="-34.4241" width="1.397" layer="16"/>
-<wire x1="61.5009" y1="-34.4241" x2="56.555" y2="-39.37" width="1.397" layer="16"/>
+<wire x1="56.555" y1="-39.37" x2="55.88" y2="-39.37" width="2.7686" layer="16"/>
+<wire x1="47.2633" y1="-8.69505" x2="49.33505" y2="-6.6233" width="2.7686" layer="16"/>
+<wire x1="55.6067" y1="-6.6233" x2="60.96" y2="-1.27" width="2.7686" layer="16"/>
+<wire x1="49.33505" y1="-6.6233" x2="55.6067" y2="-6.6233" width="2.7686" layer="16"/>
+<wire x1="47.2633" y1="-30.7533" x2="47.2633" y2="-8.69505" width="2.7686" layer="16"/>
+<wire x1="55.88" y1="-39.37" x2="47.2633" y2="-30.7533" width="2.7686" layer="16"/>
 </signal>
 <signal name="10VAC(N)">
@@
 <contactref element="R5" pad="1"/>
 <contactref element="TRANSFORMER" pad="P$3"/>
-<wire x1="46.99" y1="14.605" x2="42.545" y2="19.05" width="1.397" layer="1"/>
-<wire x1="42.545" y1="20.955" x2="42.545" y2="19.05" width="1.397" layer="1"/>
-<wire x1="46.99" y1="14.605" x2="50.8" y2="14.605" width="1.397" layer="1"/>
-<wire x1="50.8" y1="-7.8417875" x2="50.8" y2="-10.16" width="1.397" layer="1"/>
-<wire x1="50.8" y1="14.605" x2="51.6567875" y2="14.605" width="1.397" layer="1"/>
-<wire x1="54.2859" y1="11.9758875" x2="51.6567875" y2="14.605" width="1.397" layer="1"/>
-<wire x1="54.2859" y1="-4.3558875" x2="50.8" y2="-7.8417875" width="1.397" layer="1"/>
-<wire x1="54.2859" y1="11.9758875" x2="54.2859" y2="-4.3558875" width="1.397" layer="1"/>
+<wire x1="42.545" y1="20.955" x2="48.895" y2="14.605" width="2.7686" layer="1"/>
+<wire x1="48.895" y1="14.605" x2="50.8" y2="14.605" width="2.7686" layer="1"/>
+<wire x1="50.8" y1="14.605" x2="50.8" y2="12.7" width="2.7686" layer="1"/>
+<wire x1="50.8" y1="-6.27165" x2="50.8" y2="-10.16" width="2.7686" layer="1"/>
+<wire x1="50.8" y1="12.62165" x2="54.3367" y2="9.08495" width="2.7686" layer="1"/>
+<wire x1="54.3367" y1="-2.73495" x2="50.8" y2="-6.27165" width="2.7686" layer="1"/>
+<wire x1="54.3367" y1="9.08495" x2="54.3367" y2="-2.73495" width="2.7686" layer="1"/>
+<wire x1="48.895" y1="14.605" x2="50.8" y2="12.7" width="2.7686" layer="1"/>
+<wire x1="50.8" y1="12.7" x2="50.8" y2="12.62165" width="2.7686" layer="1"/>
 </signal>
 <signal name="110VAC(N)">
 <contactref element="R5" pad="2"/>
 <contactref element="110VAC(N)_OUT" pad="P$1"/>
-<wire x1="55.245" y1="-18.415" x2="57.785" y2="-18.415" width="1.397" layer="1"/>
-<wire x1="60.325" y1="-15.875" x2="57.785" y2="-18.415" width="1.397" layer="1"/>
-<wire x1="60.325" y1="-10.795" x2="60.325" y2="-15.875" width="1.397" layer="1"/>
-<wire x1="60.325" y1="-10.795" x2="60.96" y2="-10.16" width="1.397" layer="1"/>
+<wire x1="55.245" y1="-18.415" x2="60.96" y2="-12.7" width="2.7686" layer="1"/>
+<wire x1="60.96" y1="-12.7" x2="60.96" y2="-10.16" width="2.7686" layer="1"/>
 </signal>
 <signal name="110VAC(L)_OUT">
 <contactref element="SSR" pad="P$2"/>
 <contactref element="110VAC(L)_OUT" pad="P$1"/>
-<wire x1="46.355" y1="-39.37" x2="55.245" y2="-30.48" width="1.397" layer="1"/>
-<wire x1="55.245" y1="-30.48" x2="55.245" y2="-28.575" width="1.397" layer="1"/>
+<wire x1="46.355" y1="-39.37" x2="55.245" y2="-30.48" width="2.7686" layer="1"/>
+<wire x1="55.245" y1="-30.48" x2="55.245" y2="-28.575" width="2.7686" layer="1"/>
 </signal>
 <signal name="B">
